File: board/board.kicad_pcb (KiCad board)
At the start: 2 copper layers, 21 x 13 mm, 1 part

Commit message: Update PCB Design rev1.0
Parts:
- added D1: GW_J9LHS1.4M-C1C7-2+58+MQ+30A-1-100-R33, GW_J9LHS1:LED_GW_J9LHS1.4M-C1C7-2+58+MQ+30A-1-100-R33, F.Cu at (150.3, 96.5)
- added J1: 0xx_LED, on_edge:on_edge_2x05_device, F.Cu at (140.0, 96.5)
- added J2: 0xx_LED, on_edge:on_edge_2x05_host, F.Cu at (161.0, 96.5)
- LOGO1: moved to B.Cu
- moved LOGO1 0.06 mm to (150.0, 99.1), turned to 180 degrees
Routing:
- net Net-(D1-Pad7): track 0.00 -> 35.5 mm, vias 0 -> 2
- net Net-(D1-Pad4): track 0.00 -> 25.2 mm
- net Net-(D1-Pad1): track 0.00 -> 24.5 mm, vias 0 -> 2
- net Net-(D1-Pad3): track 0.00 -> 21.5 mm, vias 0 -> 2
- net Net-(D1-Pad2): track 0.00 -> 20.0 mm, vias 0 -> 2
- net (no net): vias 0 -> 88
- added copper zone on In1.Cu, net (none)
- added copper zone on In2.Cu, net (none)
Other:
- outline, holes or cut-outs redrawn
- copper layers 2 -> 4
